File: E-P-206-R2.0.0_Fuel_Cell_Controller.sch (EAGLE design)
At the start: 175 parts

Commit message: Added some silkscreening and updated the relay board connection
Parts:
- removed C1, C2: NNP, SparkFun:CAP1206
- removed C24, C26: 100nF, SparkFun:CAP0603-CAP
- removed JP1, JP4: JUMPER-31-2, SparkFun:JUMPER-31-2
- removed LD39300-NNP: LD117ADT50TR, v-reg:LD117ADT50TR
- removed R25: 10k, SparkFun-Resistors:RESISTOR-ARRAY0603-ARV
- removed R73, R86: 31.6k 1%, SparkFun:RESISTOR0603-RES
- removed R74, R76, R85: 47k 1%, SparkFun:RESISTOR0603-RES
- removed R75: 3k 1%, SparkFun:RESISTOR0603-RES
- removed U$11, U$42, U$7, U$9: (no value), diode:DIODE-DO214AC
- added R29, R56: 1M, resistor:R-US_R0805
- R15: value 3k 1% -> 1M; device SparkFun:RESISTOR0603-RES -> resistor:R-US_R0805
- R16: value 47k 1% -> 1M; device SparkFun:RESISTOR0603-RES -> resistor:R-US_R0805
Connections:
- removed net 3V: C2.1, JP1.3, JP4.3, LD39300-NNP.OUT
- removed net CAPCURR: R86.2, RJ45_0_TOP.2
- removed net CAPCURR_V_R: C26.1, JP4.2, RJ45_0_TOP.1
- removed net CAPVOLT_R: R76.1, RJ45_0_TOP.5
- removed net FCCURR: R73.2, RJ45_0_TOP.4
- removed net FCCURR_V_R: C24.1, JP1.2, RJ45_0_TOP.3
- removed net FCVOLT_R: R16.1, RJ45_0_TOP.6
- removed net N$21: MCU.PA8, R25D.1
- removed net N$27: MCU.PA9, R25C.1
- removed net N$28: MCU.PA10, R25B.1
- removed net N$29: MCU.PA11, R25A.1
- removed net N$38: MCU.PD2, U$2G$8.P$1
- new net FCC_R: RJ45_0_TOP.6
- net +12V: no longer U$11.C, U$42.C, U$7.C, U$9.C
- net CAPCURR(S): now also MCU.PA8, R15.1, RJ45_0_TOP.1; no longer R25D.2, R85.2, R86.1
- net CAPREL_R: no longer RJ45_0_BOTTOM.3, U$9.A
- net CAPVOLT: now also MCU.PA10, R29.1, RJ45_0_TOP.3; no longer R25B.2, R75.1, R76.2
- net FCCURR(S): now also MCU.PA9, R16.1, RJ45_0_TOP.2; no longer R25C.2, R73.1, R74.2
- net FCVOLT: now also MCU.PA11, R56.1, RJ45_0_TOP.4; no longer R15.1, R16.2, R25A.2
- net GND: now also R16.2, R29.2, R56.2, RJ45_0_BOTTOM.7, RJ45_0_BOTTOM.8, U$2G$10.P$1; no longer C1.2, C2.2, C24.2, C26.2, LD39300-NNP.ADJ, R74.1, R75.2, R85.1, RJ45_3_TOP.1
- net MOTORREL_R: no longer RJ45_0_BOTTOM.2, U$7.A
- net OP-1S: now also RJ45_0_BOTTOM.1
- net OP-2S: now also RJ45_0_BOTTOM.2
- net OP-3S: now also RJ45_0_BOTTOM.3
- net OP-4S: now also RJ45_0_BOTTOM.4
- net OPENLOG_TX: now also U$2G$8.P$1
- net RESREL_R: no longer RJ45_0_BOTTOM.4, U$11.A
- net STARTUPREL_R: no longer RJ45_0_BOTTOM.1, U$42.A
- net SYS_OK: now also RJ45_3_TOP.1; no longer RJ45_2_TOP.1
- net VCC: now also RJ45_0_TOP.5, U$2G$9.P$1; no longer C1.1, JP1.1, JP4.1, LD39300-NNP.IN
Other:
- note removed: "3V"
- note removed: "50v"
- note removed: "Default to +5V supply operation for sensor"
