File: E-P-206-R2.0.1 Fuel Cell Control.brd (EAGLE design)
At the start: 160 x 100 mm, 159 parts

Commit message: Second update
Parts:
- removed R29, R56: 1M, resistor:R0805
- removed U$22, U$25, U$27, U$3: (no value), SparkFun-Electromechanical:STAND-OFF
- added C1, C2: NNP, SparkFun:1206
- added C24, C25, C26: 100nF, SparkFun:0603-CAP
- added JP1, JP4: JUMPER-31-2, SparkFun:SJ_3_PASTE1&2
- added JP2: USB, SparkFun-Connectors:USB-MICROB
- added LD39300-NNP: LD117ADT50TR, v-reg:DPACK
- added R21: 4.7k, SparkFun:0603-RES
- added R25: 10k, SparkFun-Resistors:0603-ARV
- added R73, R86: 31.6k 1%, SparkFun:0603-RES
- added R74, R76, R85: 47k 1%, SparkFun:0603-RES
- added R75: 3k 1%, SparkFun:0603-RES
- added START1: 43650-0200, Shell2013:43650-0200
- added U$11, U$42, U$7, U$9: (no value), diode:DO214AC
- R15: value 1M -> 3k 1%; device resistor:R0805 -> SparkFun:0603-RES
- R16: value 1M -> 47k 1%; device resistor:R0805 -> SparkFun:0603-RES
- moved R31 126.4 mm to (38.1, 17.8)
- moved R32 120.6 mm to (40.6, 17.8)
- moved R15 8.83 mm to (76.2, 10.7)
- moved R16 5.61 mm to (77.5, 14.0), turned to 270 degrees
- moved LED7 3.81 mm to (27.9, 95.2)
- moved R10 3.79 mm to (156.2, 88.9), turned to 180 degrees
- moved R19 3.69 mm to (152.4, 88.9), turned to 0 degrees
- moved POWER 3.59 mm to (141.0, 11.4)
- moved R54 3.33 mm to (22.9, 54.6)
- moved R6 3.09 mm to (111.8, 62.2), turned to 180 degrees
- moved R34 2.54 mm to (156.2, 52.1)
- moved C19 2.54 mm to (133.3, 17.8)
- moved R35 2.54 mm to (152.4, 52.1)
- moved R3 2.47 mm to (156.2, 76.2), turned to 180 degrees
- moved R83 2.37 mm to (156.2, 96.5), turned to 0 degrees
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- renumbered U$2 to SCREWTERMINAL
Connections:
- net N$22 renamed PC21
- net N$23 renamed PC22
- net N$24 renamed PC23
- net N$30 renamed PC24
- net N$31 renamed PC31
- net N$36 renamed PD0
- removed net FCC_R: RJ45_0_.T_6
- removed net N$37: MCU.75, SCREWTERMINAL.7
- new net 3V: C2.1, JP1.3, JP4.3, LD39300-NNP.4
- new net CAPCURR: R86.2, RJ45_0_.T_2
- new net CAPCURR_V_R: C26.1, JP4.2, RJ45_0_.T_1
- new net CAPVOLT_R: R76.1, RJ45_0_.T_5
- new net FCCURR: R73.2, RJ45_0_.T_4
- new net FCCURR_V_R: C24.1, JP1.2, RJ45_0_.T_3
- new net FCVOLT_R: R16.1, RJ45_0_.T_6
- new net N$21: MCU.14, R25.4
- new net N$27: MCU.15, R25.3
- new net N$28: MCU.16, R25.2
- new net N$29: MCU.17, R25.1
- net +12V: now also U$11.C, U$42.C, U$7.C, U$9.C
- net CAPCURR(S): now also R25.5, R85.2, R86.1; no longer MCU.14, R15.1, RJ45_0_.T_1
- net CAPREL_R: now also RJ45_0_.B_3, U$9.A
- net CAPVOLT: now also R25.7, R75.1, R76.2; no longer MCU.16, R29.1, RJ45_0_.T_3
- net FCCURR(S): now also R25.6, R73.1, R74.2; no longer MCU.15, R16.1, RJ45_0_.T_2
- net FCVOLT: now also R15.1, R16.2, R25.8; no longer MCU.17, R56.1, RJ45_0_.T_4
- net GND: now also C1.2, C2.2, C24.2, C25.2, C26.2, JP2.GND, JP2.MT1, JP2.MT2, LD39300-NNP.1, R21.2, R74.1, R75.2, R85.1, RJ45_3_.T_1; no longer R16.2, R29.2, R56.2, RJ45_0_.B_7, RJ45_0_.B_8
- net MOTORREL_R: now also RJ45_0_.B_2, U$7.A
- net OP-1S: no longer RJ45_0_.B_1
- net OP-2S: no longer RJ45_0_.B_2
- net OP-3S: no longer RJ45_0_.B_3
- net OP-4S: no longer RJ45_0_.B_4
- net OPENLOG_RX: now also SCREWTERMINAL.8
- net OPENLOG_TX: now also SCREWTERMINAL.7; no longer SCREWTERMINAL.8
- net RESREL_R: now also RJ45_0_.B_4, U$11.A
- net START(S): now also C25.1, R21.1, START1.P$1
- net STARTUPREL_R: now also RJ45_0_.B_1, U$42.A
- net SYS_OK: now also RJ45_2_.T_1; no longer RJ45_3_.T_1
- net USB_N: now also JP2.D-
- net USB_P: now also JP2.D+
- net USB_VBUS: now also JP2.VBUS
- net VCC: now also C1.1, JP1.1, JP4.1, LD39300-NNP.3, START1.P$2; no longer RJ45_0_.T_5
Routing:
- net OP-3S: track 228.7 -> 2.96 mm, vias 8 -> 0
- net N$20: track 8.36 -> 190.0 mm, vias 0 -> 8
- net CAPCURR(S): track 144.3 -> 28.2 mm, vias 5 -> 2
- net FCVOLT: track 121.8 -> 7.74 mm, vias 3 -> 0
- net FCCURR(S): track 135.5 -> 25.3 mm, vias 3 -> 2
- net FCVOLT_R: track 0.00 -> 106.9 mm, vias 0 -> 4
- net CAPVOLT: track 122.4 -> 17.0 mm, vias 4 -> 2
- net FCCURR: track 0.00 -> 103.8 mm, vias 0 -> 4
- net CAPVOLT_R: track 0.00 -> 102.6 mm, vias 0 -> 4
- net CAPCURR: track 0.00 -> 100.2 mm, vias 0 -> 4
- net N$37: track 89.1 -> 0.00 mm, vias 1 -> 0
- net OPENLOG_TX: track 97.8 -> 31.5 mm, vias 3 -> 1
- net FCCURR_V_R: track 0.00 -> 51.0 mm, vias 0 -> 3
- net CAPCURR_V_R: track 0.00 -> 49.4 mm, vias 0 -> 5
- net RESREL_R: track 6.65 -> 53.9 mm, vias 0 -> 3
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Other:
- board text removed: "+12V"
- board text removed: "+5V"
- board text removed: "BTN1"
- board text removed: "BTN2"
- board text removed: "BTN3"
- board text removed: "BTN4"
- board text removed: "Fuel Cell Controller"
- board text removed: "NC"
- board text removed: "PD0"
- board text removed: "PD1"
- board text removed: "TX"
