File: E-P-206-R2.0.1 Fuel Cell Control.sch (EAGLE design)
At the start: 155 parts

Commit message: Second update
Parts:
- removed R29, R56: 1M, resistor:R-US_R0805
- removed U$2: 10X1PCBBLOCK, Shell2013:10X1PCBBLOCK
- added C1, C2: NNP, SparkFun:CAP1206
- added C24, C25, C26: 100nF, SparkFun:CAP0603-CAP
- added JP1, JP4: JUMPER-31-2, SparkFun:JUMPER-31-2
- added JP2: USB, SparkFun-Connectors:USB-MICROB
- added LD39300-NNP: LD117ADT50TR, v-reg:LD117ADT50TR
- added R21: 4.7k, SparkFun:RESISTOR0603-RES
- added R25: 10k, SparkFun-Resistors:RESISTOR-ARRAY0603-ARV
- added R73, R86: 31.6k 1%, SparkFun:RESISTOR0603-RES
- added R74, R76, R85: 47k 1%, SparkFun:RESISTOR0603-RES
- added R75: 3k 1%, SparkFun:RESISTOR0603-RES
- added SCREWTERMINAL: 10X1PCBBLOCK, Shell2013:10X1PCBBLOCK
- added START1: 43650-0200, Shell2013:43650-0200
- added U$11, U$42, U$7, U$9: (no value), diode:DIODE-DO214AC
- R15: value 1M -> 3k 1%; device resistor:R-US_R0805 -> SparkFun:RESISTOR0603-RES
- R16: value 1M -> 47k 1%; device resistor:R-US_R0805 -> SparkFun:RESISTOR0603-RES
Connections:
- removed net FCC_R: RJ45_0_TOP.6
- removed net N$22: MCU.PC21, U$2G$1.P$1
- removed net N$23: MCU.PC22, U$2G$2.P$1
- removed net N$24: MCU.PC23, U$2G$3.P$1
- removed net N$30: MCU.PC24, U$2G$4.P$1
- removed net N$31: MCU.PC31, U$2G$5.P$1
- removed net N$36: MCU.PD0, U$2G$6.P$1
- removed net N$37: MCU.PD1, U$2G$7.P$1
- new net 3V: C2.1, JP1.3, JP4.3, LD39300-NNP.OUT
- new net CAPCURR: R86.2, RJ45_0_TOP.2
- new net CAPCURR_V_R: C26.1, JP4.2, RJ45_0_TOP.1
- new net CAPVOLT_R: R76.1, RJ45_0_TOP.5
- new net FCCURR: R73.2, RJ45_0_TOP.4
- new net FCCURR_V_R: C24.1, JP1.2, RJ45_0_TOP.3
- new net FCVOLT_R: R16.1, RJ45_0_TOP.6
- new net N$21: MCU.PA8, R25D.1
- new net N$27: MCU.PA9, R25C.1
- new net N$28: MCU.PA10, R25B.1
- new net N$29: MCU.PA11, R25A.1
- new net PC21: MCU.PC21, SCREWTERMINALG$1.P$1
- new net PC22: MCU.PC22, SCREWTERMINALG$2.P$1
- new net PC23: MCU.PC23, SCREWTERMINALG$3.P$1
- new net PC24: MCU.PC24, SCREWTERMINALG$4.P$1
- new net PC31: MCU.PC31, SCREWTERMINALG$5.P$1
- new net PD0: MCU.PD0, SCREWTERMINALG$6.P$1
- net +12V: now also U$11.C, U$42.C, U$7.C, U$9.C
- net CAPCURR(S): now also R25D.2, R85.2, R86.1; no longer MCU.PA8, R15.1, RJ45_0_TOP.1
- net CAPREL_R: now also RJ45_0_BOTTOM.3, U$9.A
- net CAPVOLT: now also R25B.2, R75.1, R76.2; no longer MCU.PA10, R29.1, RJ45_0_TOP.3
- net FCCURR(S): now also R25C.2, R73.1, R74.2; no longer MCU.PA9, R16.1, RJ45_0_TOP.2
- net FCVOLT: now also R15.1, R16.2, R25A.2; no longer MCU.PA11, R56.1, RJ45_0_TOP.4
- net GND: now also C1.2, C2.2, C24.2, C25.2, C26.2, JP2.GND, LD39300-NNP.ADJ, R21.2, R74.1, R75.2, R85.1, RJ45_3_TOP.1, SCREWTERMINALG$10.P$1; no longer R16.2, R29.2, R56.2, RJ45_0_BOTTOM.7, RJ45_0_BOTTOM.8, U$2G$10.P$1
- net MOTORREL_R: now also RJ45_0_BOTTOM.2, U$7.A
- net OP-1S: no longer RJ45_0_BOTTOM.1
- net OP-2S: no longer RJ45_0_BOTTOM.2
- net OP-3S: no longer RJ45_0_BOTTOM.3
- net OP-4S: no longer RJ45_0_BOTTOM.4
- net OPENLOG_RX: now also SCREWTERMINALG$8.P$1
- net OPENLOG_TX: now also SCREWTERMINALG$7.P$1; no longer U$2G$8.P$1
- net RESREL_R: now also RJ45_0_BOTTOM.4, U$11.A
- net START(S): now also C25.1, R21.1, START1.P$2
- net STARTUPREL_R: now also RJ45_0_BOTTOM.1, U$42.A
- net SYS_OK: now also RJ45_2_TOP.1; no longer RJ45_3_TOP.1
- net USB_N: now also JP2.D-
- net USB_P: now also JP2.D+
- net USB_VBUS: now also JP2.VBUS
- net VCC: now also C1.1, JP1.1, JP4.1, LD39300-NNP.IN, SCREWTERMINALG$9.P$1, START1.P$1; no longer RJ45_0_TOP.5, U$2G$9.P$1
Other:
- note added: "3V"
- note added: "50v"
- note added: "Default to +5V supply operation for sensor"
- note added: "USB Port"
- moved on the sheet: R15, R16, R6
